File: hardware/Servo.brd (EAGLE design)
At the start: 45.7 x 58.2 mm, 25 parts, among them Q2 IRLML6401

Commit message: Hardware V4.0
Other:
- board text added: "Servo-Dekoder Aufsatz V4.0 für Basisplatine 3.0 (saaralf)"
- board text removed: "Servo-Dekoder Aufsatz V1.0"
Changed lines of the file:
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@@
 <wire x1="45.72" y1="58.42" x2="0" y2="58.42" width="0.254" layer="20"/>
 <wire x1="0" y1="58.42" x2="0" y2="0.254" width="0.254" layer="20"/>
-<text x="35.052" y="57.15" size="1.778" layer="25" font="vector" ratio="12" rot="R180">Servo-Dekoder
-Aufsatz V1.0</text>
+<text x="13.462" y="29.464" size="1.778" layer="25" font="vector" ratio="12" rot="R270">Servo-Dekoder
+Aufsatz V4.0 für
+Basisplatine 3.0
+(saaralf)</text>
 <text x="41.402" y="2.794" size="1.27" layer="16" font="vector" ratio="12" rot="MR180">BOT</text>
 <dimension x1="0" y1="58.42" x2="45.72" y2="58.42" x3="22.86" y3="60.706" textsize="1.778" layer="16"/>
