File: hardware/Servo.sch (EAGLE design)
At the start: 25 parts, among them Q2 IRLML6401

Commit message: Hardware V4.0
Other:
- note added: "FunktionsdekoderAufsatz V4.0 für openSX (saaralf) Basisplatine V3.0"
- note removed: "FunktionsdekoderAufsatz V3.2 für openSX Basisplatine 2.0"
Changed lines of the file:
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@@
 saaralf Modellbahn</text>
 <text x="175.26" y="2.54" size="1.778" layer="101">23.10.2024</text>
-<text x="180.34" y="20.32" size="1.778" layer="101">FunktionsdekoderAufsatz V3.2 für openSX Basisplatine 2.0</text>
+<text x="180.34" y="20.32" size="1.778" layer="101">FunktionsdekoderAufsatz V4.0 für openSX (saaralf) Basisplatine V3.0</text>
 <text x="106.68" y="48.26" size="1.778" layer="97">Reverse voltage</text>
 <text x="109.22" y="45.72" size="1.778" layer="97">protection</text>
